File: Sema/schematic.kicad_pcb (KiCad board)
At the start: 2 copper layers, 100 x 93 mm, 95 parts, among them J1 Conn_01x05_Male, J10 Conn_01x05_Male, J11 Conn_01x05_Male, J12 Conn_01x05_Male, J13 Conn_01x01_Male, J14 Conn_01x01_Male, J15 Conn_01x01_Male, J16 Conn_01x01_Male, J2 Conn_01x01_Male, J3 Conn_01x03_Male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

Commit message: Final version
Connections:
- U5 pad 4: unconnected-(U5-Pad4) -> 3.3V
Routing:
- net 3.3V: track 473.9 -> 481.8 mm
