File: Sema/schematic.kicad_sch (KiCad schematic)
At the start: 91 parts, among them U1 SN74LS75DR, U2 SN74LS75DR, U3 SN74LS75DR, U3.3V LM317BTG, U4 SN74LS75DR, U5 SN74LS75DR, U5V LM317BTG, U6 SN74LS75DR

Commit message: Rutiran PCB Prepravljena šema u skladu sa zahtjevima
Parts:
- removed 0.1uF, 1uF: 08055A220JAT2A, CAP_0805J_AVX, symbol 2022-12-14_18-04-28:08055A220JAT2A
- removed 1k, 3k: HCJ0805ZT0R00, STA_HCJ0805_STP, symbol HCJ0805ZT0R00:HCJ0805ZT0R00
- removed A? (x6): PINK, symbol Connector:TestPoint
- removed CS, MCLR*, MISO, MOSI/SDA, PGC, PGD, SCLK/SCL, VDD, VSS: TestPoint_Small, symbol Connector:TestPoint_Small
- removed GND (x2), RX, TX, VCC3.3V, YELLOW, YELLOW? (x5): TestPoint, symbol Connector:TestPoint
- removed JP1: Jumper_3_Bridged12, symbol Jumper:Jumper_3_Bridged12
- removed TX? (x6), Vin: 12V, symbol Connector:TestPoint
- removed TX? (x6): ORANGE, symbol Connector:TestPoint
- removed TX? (x6): BLUE, symbol Connector:TestPoint
- removed U1, U2, U3, U4, U5, U6: SN74LS75DR, D16, symbol SN74LS75DR:SN74LS75DR
- removed U5V: LM317BTG, TO-220AB_ONS, symbol LM317BTG:LM317BTG
- added 0.1uF1: 08055A220JAT2A, footprints:08055A220JAT2A, symbol 2022-12-14_18-04-28:08055A220JAT2A
- added C11, C12, C13, C14, C15, C16, C17, C18, C19, C4, C7, C8: 0.1uF, footprints:08055A220JAT2A, symbol 2022-12-14_18-04-28:08055A220JAT2A
- added H1, H2, H3, H4: MountingHole, MountingHole:MountingHole_2.5mm, symbol Mechanical:MountingHole
- added J1, J10, J2, J5, J6, J7, J8, J9: Conn_01x05_Male, Connector_PinHeader_1.00mm:PinHeader_1x05_P1.00mm_Vertical, symbol Connector:Conn_01x05_Male
- added J11, J12: Conn_01x03_Male, Connector_PinHeader_1.00mm:PinHeader_1x03_P1.00mm_Vertical, symbol Connector:Conn_01x03_Male
- added J3: Conn_01x02_Male, Connector_PinHeader_1.00mm:PinHeader_1x02_P1.00mm_Vertical, symbol Connector:Conn_01x02_Male
- added J4: USB_B, Connector_USB:USB_B_TE_5787834_Vertical, symbol Connector:USB_B
- added R14, R8: 10k, HCJ0805ZT0R00j:HCJ0805ZT0R00, symbol HCJ0805ZT0R00:HCJ0805ZT0R00
- added R9: 14k, HCJ0805ZT0R00j:HCJ0805ZT0R00, symbol HCJ0805ZT0R00:HCJ0805ZT0R00
- added U10, U5, U6, U7, U8, U9: 74LVT573MTC, 74LVT573MTCj:74LVT573MTC, symbol 74LVT573MTC:74LVT573MTC
- added U3: FT232RL, Package_SO:SSOP-28_5.3x10.2mm_P0.65mm, symbol Interface_USB:FT232RL
- C1, C2: renamed from 22pF; value 08055A220JAT2A -> 22pF; footprint CAP_0805J_AVX -> footprints:08055A220JAT2A
- C10: renamed from 10uF; value 08055A220JAT2A -> 10uF; footprint CAP_0805J_AVX -> footprints:08055A220JAT2A
- C3, C9: renamed from 0.1uF; value 08055A220JAT2A -> 0.1uF; footprint CAP_0805J_AVX -> footprints:08055A220JAT2A
- C5: renamed from 1uF; value 08055A220JAT2A -> 22uf; footprint CAP_0805J_AVX -> footprints:08055A220JAT2A
- C6: renamed from 0.1uF; value 08055A220JAT2A -> 22uF; footprint CAP_0805J_AVX -> footprints:08055A220JAT2A
- R1, R2, R6, R7: renamed from 10k; value HCJ0805ZT0R00 -> 10k; footprint STA_HCJ0805_STP -> HCJ0805ZT0R00j:HCJ0805ZT0R00
- R10, R11, R12, R13: renamed from 10k?; value HCJ0805ZT0R00 -> 10k; footprint STA_HCJ0805_STP -> HCJ0805ZT0R00j:HCJ0805ZT0R00
- R3: renamed from 12k; value HCJ0805ZT0R00 -> 12k; footprint STA_HCJ0805_STP -> HCJ0805ZT0R00j:HCJ0805ZT0R00
- R4: renamed from 0.3k; value HCJ0805ZT0R00 -> 300; footprint STA_HCJ0805_STP -> HCJ0805ZT0R00j:HCJ0805ZT0R00
- R5: renamed from 7.5k; value HCJ0805ZT0R00 -> 7.5k; footprint STA_HCJ0805_STP -> HCJ0805ZT0R00j:HCJ0805ZT0R00
- TP1.1, TP1.2, TP2.1, TP2.2, TP3.1, TP3.2, TP4.1, TP4.2: footprint (none) -> MountingHole:MountingHole_2.2mm_M2_DIN965_Pad
- U1: renamed from U?; footprint SOIC28__SO28_MCH -> PIC24FJ64GA702-ISO:PIC24FJ64GA702-I&slash_SO
- U11, U12, U13, U14: renamed from U?; footprint D16 -> ULN2003AIDRj:ULN2003AIDR
- U2: renamed from U?; footprint ABLS-8.000MHZ-B2-T_ABR -> ABLS-8:ABLS-8.000MHZ-B2-T
- U3.3V1: renamed from U3.3V; footprint TO-220AB_ONS -> LM317BTGj:LM317BTG
- U4: renamed from U?; footprint DW0024A_N -> CD74HC4514M96j:CD74HC4514M96
Connections:
- net 12V: now also C16.2, C17.2, C18.2, C19.2, J10.1 (Pin_1), J3.1 (Pin_1), J5.1 (Pin_1), J6.1 (Pin_1), J7.1 (Pin_1), J8.1 (Pin_1), J9.1 (Pin_1), R9.1
- net 3.3V: now also 0.1uF1.2, C11.2, C12.2, C13.2, C14.2, C15.2, C8.1, J11.3 (Pin_3), J2.2 (Pin_2), R14.1, U10.20 (VCC), U5.20 (VCC), U6.20 (VCC), U7.20 (VCC), U8.20 (VCC), U9.20 (VCC)
- net 5V: now also J4.1 (VBUS), R8.2, R9.2, U3.20 (VCC)
- net D1: now also U1.24 (AN7/C1INC/RP13/OCM1D/CTPLS/RB13), U10.2 (D0), U5.2 (D0), U6.2 (D0), U7.2 (D0), U8.2 (D0), U9.2 (D0); no longer U1.26 (AN9/C3INA/RP15/CTED6/RB15)
- net D2: now also U1.23 (AN8/LVDIN/RP12/RB12), U10.3 (D1), U5.3 (D1), U6.3 (D1), U7.3 (D1), U8.3 (D1), U9.3 (D1); no longer U1.25 (CVREF/AN6/C3INB/RP14/CTED5/RB14)
- net D3: now also U1.22 (PGC2/TMS/REFI1/RP11/CTED9/RB11), U10.4 (D2), U5.4 (D2), U6.4 (D2), U7.4 (D2), U8.4 (D2), U9.4 (D2); no longer U1.24 (AN7/C1INC/RP13/OCM1D/CTPLS/RB13)
- net D4: now also U1.21 (PGD2/TDI/RP10/OCM1C/CTED11/RB10), U10.5 (D3), U5.5 (D3), U6.5 (D3), U7.5 (D3), U8.5 (D3), U9.5 (D3); no longer U1.23 (AN8/LVDIN/RP12/RB12)
- net E1: now also U5.11 (LE)
- net E2: now also U6.11 (LE)
- net E3: now also U7.11 (LE)
- net E4: now also U8.11 (LE)
- net E5: now also U9.11 (LE)
- net E6: now also U10.11 (LE)
- net GND: now also U1.19 (VSS), 0.1uF1.1, C11.1, C12.1, C13.1, C14.1, C15.1, C16.1, C17.1, C18.1, C19.1, C4.2, C7.1, C8.2, J1.5 (Pin_5), J2.3 (Pin_3), J3.2 (Pin_2), J4.4 (GND), R8.1, U10.1 (OE_N), U10.10 (GND), U10.6 (D4), U10.7 (D5), U10.8 (D6), U10.9 (D7), U3.18 (GND), U3.21 (GND), U3.25 (AGND), U3.26 (TEST), U3.7 (GND), U5.1 (OE_N), U5.10 (GND), U5.6 (D4), U5.7 (D5), U5.8 (D6), U5.9 (D7), U6.1 (OE_N), U6.10 (GND), U6.6 (D4), U6.7 (D5), U6.8 (D6), U6.9 (D7), U7.1 (OE_N), U7.10 (GND), U7.6 (D4), U7.7 (D5), U7.8 (D6), U7.9 (D7), U8.1 (OE_N), U8.10 (GND), U8.6 (D4), U8.7 (D5), U8.8 (D6), U8.9 (D7), U9.1 (OE_N), U9.10 (GND), U9.6 (D4), U9.7 (D5), U9.8 (D6), U9.9 (D7)
- net P1: now also U1.7 (AN5/C1INA/RP3/SCL2/CTED8/RB3); no longer U1.18 (TDO/C1INC/C2INC/C3INC/TMPRN/RP9/SDA1/T1CK/CTED4/RB9)
- net P2: now also U1.11 (SOSCI/RP4/RB4); no longer U1.7 (AN5/C1INA/RP3/SCL2/CTED8/RB3)
- net P3: now also U1.12 (SOSCO/PWRLCLK/RA4); no longer U1.11 (SOSCI/RP4/RB4)
- net P4: now also U1.14 (PGD3/RP5/ASDA1/OCM1E/RB5); no longer U1.12 (SOSCO/PWRLCLK/RA4)
- net Q1.1: now also U5.19 (O0)
- net Q1.2: now also U6.19 (O0)
- net Q1.3: now also U7.19 (O0)
- net Q1.4: now also U8.19 (O0)
- net Q1.5: now also U9.19 (O0)
- net Q1.6: now also U10.19 (O0)
- net Q2.1: now also U5.18 (01)
- net Q2.2: now also U6.18 (01)
- net Q2.3: now also U7.18 (01)
- net Q2.4: now also U8.18 (01)
- net Q2.5: now also U9.18 (01)
- net Q2.6: now also U10.18 (01)
- net Q3.1: now also U5.17 (02)
- net Q3.2: now also U6.17 (02)
- net Q3.3: now also U7.17 (02)
- net Q3.4: now also U8.17 (02)
- net Q3.5: now also U9.17 (02)
- net Q3.6: now also U10.17 (02)
- net Q4.1: now also U5.16 (03)
- net Q4.2: now also U6.16 (03)
- net Q4.3: now also U7.16 (03)
- net Q4.4: now also U8.16 (03)
- net Q4.5: now also U9.16 (03)
- net Q4.6: now also U10.16 (03)
- net Y6: now reaches U14.16 (1C)
- net Y6: now also J9.3 (Pin_3)
- net PI2: now reaches U11.10 (7C)
- net PI2: now also J6.4 (Pin_4)
- net Y2: now reaches U11.11 (6C)
- net Y2: now also J6.3 (Pin_3)
- net O2: now reaches U11.12 (5C)
- net O2: now also J6.2 (Pin_2)
- net B1: now reaches U11.13 (4C)
- net B1: now also J5.5 (Pin_5)
- net PI1: now reaches U11.14 (3C)
- net PI1: now also J5.4 (Pin_4)
- net Y1: now reaches U11.15 (2C)
- net Y1: now also J5.3 (Pin_3)
- net O1: now reaches U11.16 (1C)
- net O1: now also J5.2 (Pin_2)
- net Y3: now reaches U12.14 (3C)
- net Y3: now also J7.3 (Pin_3)
- net PGC: now reaches R6.1
- net PGC: now also U1.26 (AN9/C3INA/RP15/CTED6/RB15), J2.5 (Pin_5); no longer U1.5 (PGC1/AN1-/AN3/C2INA/RP1/CTED12/RB1)
- net Y4: now reaches U12.10 (7C)
- net Y4: now also J10.3 (Pin_3)
- net O4: now reaches U12.11 (6C)
- net O4: now also J10.2 (Pin_2)
- net B3: now reaches U12.12 (5C)
- net B3: now also J7.5 (Pin_5)
- net PI3: now reaches U12.13 (4C)
- net PI3: now also J7.4 (Pin_4)
- net O3: now reaches U12.15 (2C)
- net O3: now also J7.2 (Pin_2)
- net B2: now reaches U12.16 (1C)
- net B2: now also J6.5 (Pin_5)
- net OSCI: now reaches C1.2, U1.9 (OSCI/CLKI/C1IND/RA2), U2.1
- net OSCO: now reaches C2.2, U1.10 (OSCO/CLKO/C2IND/RA3), U2.2
- net O5: now reaches U13.14 (3C)
- net O5: now also J8.2 (Pin_2)
- net PI5: now reaches U13.12 (5C)
- net PI5: now also J8.4 (Pin_4)
- net B6: now reaches U14.14 (3C)
- net B6: now also J9.5 (Pin_5)
- net A0: now reaches U4.2 (A0)
- net A0: now also U1.17 (TCK/RP8/SCL1/OCM1B/CTED10/RB8); no longer U1.15 (PGC3/RP6/ASCL1/OCM1F/RB6)
- net A2: now reaches U4.21 (A2)
- net A2: now also U1.15 (PGC3/RP6/ASCL1/OCM1F/RB6); no longer U1.17 (TCK/RP8/SCL1/OCM1B/CTED10/RB8)
- net A1: now reaches U1.16 (RP7/OCM1A/CTED3/INT0/RB7), U4.3 (A1)
- net PI6: now reaches U14.15 (2C)
- net PI6: now also J9.4 (Pin_4)
- net at U1.1 (*MCLR): now also J11.2 (Pin_2), J12.1 (Pin_1)
- net SCL: now reaches R1.2, U1.2 (VREF+/CVREF+/AN0/C3INC/RP26/CTED1/RA0)
- net SCL: now also J1.1 (Pin_1)
- net MISO: now reaches U1.4 (PGD1/AN2/CTCMP/C2INB/RP0/RB0)
- net MISO: now also J1.3 (Pin_3); no longer R7.1
- net PI4: now reaches U13.16 (1C)
- net PI4: now also J10.4 (Pin_4)
- net B4: now reaches U13.15 (2C)
- net B4: now also J10.5 (Pin_5)
- net Y5: now reaches U13.13 (4C)
- net Y5: now also J8.3 (Pin_3)
- net MOSI: now reaches R2.2, U1.3 (VREF-/CVREF-/AN1/C3IND/RP27/CTED2/RA1)
- net MOSI: now also J1.2 (Pin_2)
- net RX: now reaches U1.6 (AN4/C1INB/RP2/SDA2/CTED13/RB2)
- net RX: now also U3.1 (TXD)
- net B5: now reaches U13.11 (6C)
- net B5: now also J8.5 (Pin_5)
- net O6: now reaches U13.10 (7C)
- net O6: now also J9.2 (Pin_2)
- new net: J11.1 (Pin_1), J2.1 (Pin_1)
- new net: J12.3 (Pin_3), R14.2
- new net: C7.2, U3.17 (3V3OUT)
- new net: C4.1, J12.2 (Pin_2)
- new net CS: J1.4 (Pin_4), U1.18 (TDO/C1INC/C2INC/C3INC/TMPRN/RP9/SDA1/T1CK/CTED4/RB9)
- new net D+: J4.3 (D+), U3.15 (USBD+)
- new net D-: J4.2 (D-), U3.16 (USBD-)
- new net PGD: J2.4 (Pin_4), R7.1, U1.25 (CVREF/AN6/C3INB/RP14/CTED5/RB14)
- new net tx: U1.5 (PGC1/AN1-/AN3/C2INA/RP1/CTED12/RB1), U3.5 (RXD)
Other:
- moved on the sheet: C10, C3, R10, R11, R12, R13, R6, R7, TP1.1, TP1.2, TP2.1, TP2.2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

Commit message: Dodat peti prekidac i u folderu Datasheet komponenti dodat datasheet koristenog multipleksera
Parts:
- added R?: 10k, HCJ0805ZT0R00j:HCJ0805ZT0R00, symbol HCJ0805ZT0R00:HCJ0805ZT0R00
- added TP5.1, TP5.2: TestPoint_Small, MountingHole:MountingHole_2.2mm_M2_DIN965_Pad, symbol Connector:TestPoint_Small
- added U?: PTMUX1308QDYYRQ1, SOT_8QDYYRQ1_TEX, symbol 2023-01-18_13-22-56:PTMUX1308QDYYRQ1
Connections:
- net 3.3V: now also TP5.2.1, U?.16 (VDD)
- net GND: now also R?.1, U?.2 (S6), U?.4 (S7), U?.5 (S5), U?.6 (EN), U?.8 (GND)
- net MISO: now also U1.11 (SOSCI/RP4/RB4); no longer U1.4 (PGD1/AN2/CTCMP/C2INB/RP0/RB0)
- net P1: now also U?.13 (S0); no longer U1.7 (AN5/C1INA/RP3/SCL2/CTED8/RB3)
- net P2: now also U?.14 (S1); no longer U1.11 (SOSCI/RP4/RB4)
- net P3: now also U?.15 (S2); no longer U1.12 (SOSCO/PWRLCLK/RA4)
- net P4: now also U?.12 (S3); no longer U1.14 (PGD3/RP5/ASDA1/OCM1E/RB5)
- net PGC: now also U1.5 (PGC1/AN1-/AN3/C2INA/RP1/CTED12/RB1); no longer U1.26 (AN9/C3INA/RP15/CTED6/RB15)
- net PGD: now also U1.4 (PGD1/AN2/CTCMP/C2INB/RP0/RB0); no longer U1.25 (CVREF/AN6/C3INB/RP14/CTED5/RB14)
- net RX: now also U1.7 (AN5/C1INA/RP3/SCL2/CTED8/RB3); no longer U1.6 (AN4/C1INB/RP2/SDA2/CTED13/RB2)
- net tx: now also U1.6 (AN4/C1INB/RP2/SDA2/CTED13/RB2); no longer U1.5 (PGC1/AN1-/AN3/C2INA/RP1/CTED12/RB1)
- new net M: U1.26 (AN9/C3INA/RP15/CTED6/RB15), U?.3 (D)
- new net P5: R?.2, TP5.1.1, U?.1 (S4)
- new net S0: U1.25 (CVREF/AN6/C3INB/RP14/CTED5/RB14), U?.11 (A0)
- new net S1: U1.12 (SOSCO/PWRLCLK/RA4), U?.10 (A1)
- new net S2: U1.14 (PGD3/RP5/ASDA1/OCM1E/RB5), U?.9 (A2)
Other:
- moved on the sheet: 0.1uF1, C11, C12, C13, C14, C15, C16, C17, C18, C19, C7, J10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

Commit message: Dodat bajpas kondezator na ulaze za napajanje multipleksera
Parts:
- added C?: 0.1uF, footprints:08055A220JAT2A, symbol 2022-12-14_18-04-28:08055A220JAT2A
Connections:
- net 3.3V: now also C?.2
- net GND: now also C?.1
Changed lines of the file:
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@@
   (junction (at 57.15 113.03) (diameter 0) (color 0 0 0 0)
   )
+  (junction (at 317.5 71.12) (diameter 0) (color 0 0 0 0)
+  )
   (junction (at 347.98 383.54) (diameter 0) (color 0 0 0 0)
   )
@@
     (stroke (width 0) (type default) (color 0 0 0 0))
   )
+  (wire (pts (xy 317.5 71.12) (xy 318.77 71.12))
+    (stroke (width 0) (type default) (color 0 0 0 0))
+  )
   (wire (pts (xy 443.23 210.82) (xy 453.39 210.82))
     (stroke (width 0) (type default) (color 0 0 0 0))
@@
     (stroke (width 0) (type default) (color 0 0 0 0))
   )
-  (wire (pts (xy 313.69 71.12) (xy 318.77 71.12))
+  (wire (pts (xy 313.69 71.12) (xy 317.5 71.12))
     (stroke (width 0) (type default) (color 0 0 0 0))
   )
@@
     (stroke (width 0) (type default) (color 0 0 0 0))
   )
+  (wire (pts (xy 317.5 83.82) (xy 317.5 71.12))
+    (stroke (width 0) (type default) (color 0 0 0 0))
+  )
   (wire (pts (xy 193.04 238.76) (xy 201.93 238.76))
     (stroke (width 0) (type default) (color 0 0 0 0))
   )
+  (wire (pts (xy 365.76 83.82) (xy 365.76 53.34))
+    (stroke (width 0) (type default) (color 0 0 0 0))
+  )
   (wire (pts (xy 302.26 30.48) (xy 300.99 30.48))
     (stroke (width 0) (type default) (color 0 0 0 0))
@@
     (stroke (width 0) (type default) (color 0 0 0 0))
   )
-  (wire (pts (xy 360.68 53.34) (xy 359.41 53.34))
+  (wire (pts (xy 359.41 53.34) (xy 365.76 53.34))
     (stroke (width 0) (type default) (color 0 0 0 0))
   )
@@
     (stroke (width 0) (type default) (color 0 0 0 0))
   )
+  (wire (pts (xy 334.01 83.82) (xy 317.5 83.82))
+    (stroke (width 0) (type default) (color 0 0 0 0))
+  )
   (wire (pts (xy 394.97 255.27) (xy 402.59 255.27))
     (stroke (width 0) (type default) (color 0 0 0 0))
@@
     (stroke (width 0) (type default) (color 0 0 0 0))
   )
+  (wire (pts (xy 341.63 83.82) (xy 365.76 83.82))
+    (stroke (width 0) (type default) (color 0 0 0 0))
+  )
   (wire (pts (xy 245.11 162.56) (xy 254 162.56))
     (stroke (width 0) (type default) (color 0 0 0 0))
@@
     (pin "2")
   )
+  (symbol (lib_id "2022-12-14_18-04-28:08055A220JAT2A") (at 334.01 83.82 0) (unit 1)
+    (in_bom yes) (on_board yes)
+    (property "Reference" "C?" (id 0) (at 335.28 80.01 0)
+      (effects (font (size 1.524 1.524)) (justify left))
+    )
+    (property "Value" "0.1uF" (id 1) (at 328.93 87.63 0)
+      (effects (font (size 1.524 1.524)) (justify left))
+    )
+    (property "Footprint" "footprints:08055A220JAT2A" (id 2) (at 337.82 92.964 0)
+      (effects (font (size 1.524 1.524)) hide)
+    )
+    (property "Datasheet" "" (id 3) (at 334.01 83.82 0)
+      (effects (font (size 1.524 1.524)))
+    )
+    (pin "1")
+    (pin "2")
+  )
   (symbol (lib_id "power:GND") (at 58.42 124.46 0) (unit 1)
     (in_bom yes) (on_board yes) (fields_autoplaced)
@@
       (reference "C19") (unit 1) (value "0.1uF") (footprint "footprints:08055A220JAT2A")
     )
+    (path "/e453a314-d67e-4927-b098-3b8ec0b104e3"
+      (reference "C?") (unit 1) (value "0.1uF") (footprint "footprints:08055A220JAT2A")
+    )
     (path "/14bd4efb-f471-4ac6-865a-a60d9f817d90"

Commit message: Finalna verzija layout-a
Parts:
- removed R8: 10k, HCJ0805ZT0R00j:HCJ0805ZT0R00, symbol HCJ0805ZT0R00:HCJ0805ZT0R00
- removed R9: 14k, HCJ0805ZT0R00j:HCJ0805ZT0R00, symbol HCJ0805ZT0R00:HCJ0805ZT0R00
- removed U3.3V1: LM317BTG, LM317BTGj:LM317BTG, symbol LM317BTG:LM317BTG
- added C1: 0.1uF, footprints:08055A220JAT2A, symbol 2022-12-14_18-04-28:08055A220JAT2A
- added C2: 100uF, footprints:08055A220JAT2A, symbol 2022-12-14_18-04-28:08055A220JAT2A
- added R4: 820, HCJ0805ZT0R00j:HCJ0805ZT0R00, symbol HCJ0805ZT0R00:HCJ0805ZT0R00
- added U1, U2: LM317AT/NOPB, LM317AT:LM317AT, symbol LM317AT&slash_NOPB:LM317AT/NOPB
- C7: renamed from C5; value 22uf -> 100uf
- C8: renamed from C6; value 22uF -> 0.1uF
- H1, H2, H3, H4: footprint MountingHole:MountingHole_2.5mm -> MountingHole:MountingHole_3.5mm
- R3: value 12k -> 270
- TP1.1, TP1.2, TP2.1, TP2.2, TP3.1, TP3.2, TP4.1, TP4.2, TP5.1, TP5.2: footprint MountingHole:MountingHole_2.2mm_M2_DIN965_Pad -> Connector_PinHeader_1.00mm:PinHeader_1x01_P1.00mm_Vertical
- U7: renamed from U?; footprint SOT_8QDYYRQ1_TEX -> PTMUX1308QDYYRQ1j:PTMUX1308QDYYRQ1
- gave numbers to parts that had none: 2
- renumbered C8 to C10, C9 to C11, C10 to C12, C11 to C14, C12 to C15, C13 to C16, C14 to C17, C15 to C18, C16 to C19, C17 to C20, C18 to C21, C19 to C22, C1 to C3, C2 to C4, C3 to C5, C4 to C6, C7 to C9, J8 to J10, J9 to J11, J10 to J12, J3 to J2, J11 to J3, J2 to J4, J12 to J5, J4 to J6, J5 to J7, J6 to J8, J7 to J9, R4 to R5, R5 to R6, R14 to R7, R6 to R8, R7 to R9, U7 to U10, U8 to U11, U9 to U12, U10 to U13, U11 to U14, U12 to U15, U13 to U16, U14 to U17, U1 to U3, U2 to U4, U3 to U5, U4 to U6, U5 to U8, U6 to U9
Connections:
- net 12V: now also C1.1, U1.3 (IN), U2.3 (IN)
- net 3.3V: now also U2.2 (OUT)
- net 5V: now also R3.2, C2.2, U1.2 (OUT)
- net GND: now also R5.1, C1.2, C2.1, R4.1; no longer R3.2
- net at R3.1: now also R4.2, U1.1 (ADJ); no longer R5.1
- net at R5.2, R6.1: now also U2.1 (ADJ)

Commit message: Izmjene na layout-u
Parts:
- removed J2: Conn_01x02_Male, Connector_PinHeader_1.00mm:PinHeader_1x02_P1.00mm_Vertical, symbol Connector:Conn_01x02_Male
- added J13, J14, J15, J16, J2: Conn_01x01_Male, Connector_PinHeader_1.00mm:PinHeader_1x01_P1.00mm_Vertical, symbol Connector:Conn_01x01_Male
- added TP1, TP10, TP11, TP2, TP3, TP4, TP5, TP6, TP7, TP8, TP9: TestPoint, Connector_PinHeader_1.00mm:PinHeader_1x01_P1.00mm_Vertical, symbol Connector:TestPoint
Connections:
- net 12V: now also J2.1 (Pin_1)
- net 3.3V: now also TP3.1
- net 5V: now also TP1.1
- net E1: now also TP6.1
- net E2: now also TP7.1
- net E3: now also TP8.1
- net E4: now also TP9.1
- net E5: now also TP10.1
- net E6: now also TP11.1
- net GND: now also J13.1 (Pin_1), J14.1 (Pin_1), J15.1 (Pin_1), J16.1 (Pin_1)
- net RX: now also TP5.1
- net tx: now also TP4.1
- net at J3.2 (Pin_2), J5.1 (Pin_1), U3.1 (*MCLR): now also TP2.1

Commit message: Final version
Connections:
- net 3.3V: now also U5.4 (VCCIO)
Changed lines of the file:
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@@
+    )
+  )
+  (global_label "3.3V" (shape input) (at 219.71 20.32 90) (fields_autoplaced)
+    (effects (font (size 1.27 1.27)) (justify left))
+    (property "Intersheet References" "${INTERSHEET_REFS}" (id 0) (at 219.7894 13.7945 90)
+      (effects (font (size 1.27 1.27)) (justify left) hide)
     )
   )
